File: Hardware/KiCad/FritzRT.sch (KiCad schematic (older format))
At the start: 2 parts

Commit message: Added new part
Parts:
- added AT? (x2): 10dB, symbol ATTENUATOR
- added U? (x2): PE42421, symbol PE42421
Connections:
- new net: AT?.1, AT?.3
- new net: AT?.3, U?.1 (RF1)
- new net: AT?.1, U?.1 (RF1)
- new net: U?.3 (RF2), U?.3 (RF2)
- new net GND: AT?.2, AT?.2, U?.2 (GND), U?.2 (GND)
Changed lines of the file:
@@
 LIBS:FritzLib
 LIBS:FritzLib2
-EELAYER 25 0
+LIBS:FritzRT-cache
+EELAYER 26 0
 EELAYER END
 $Descr A3 16535 11693
@@
 P 3150 4200
 F 0 "U?" H 1500 5850 50  0000 C CNN
-F 1 "SAMD20G18A-MU" H 4600 2550 50  0000 C CNN
+F 1 "SAMD20G18A-MU" H 4525 5850 50  0000 C CNN
 F 2 "QFN48" H 3150 3050 50  0001 C CIN
 F 3 "" H 3150 4450 50  0001 C CNN
@@
 	1    0    0    -1
 $EndComp
+$Comp
+L ATTENUATOR AT?
+U 1 1 595ED8CC
+P 6875 7050
+F 0 "AT?" V 6668 7050 50  0000 C CNN
+F 1 "10dB" V 6759 7050 50  0000 C CNN
+F 2 "" H 6875 7050 50  0001 C CNN
+F 3 "" H 6875 7050 50  0001 C CNN
+	1    6875 7050
+	0    1    1    0
+$EndComp
+$Comp
+L ATTENUATOR AT?
+U 1 1 595EDAA0
+P 7275 7050
+F 0 "AT?" V 7068 7050 50  0000 C CNN
+F 1 "10dB" V 7159 7050 50  0000 C CNN
+F 2 "" H 7275 7050 50  0001 C CNN
+F 3 "" H 7275 7050 50  0001 C CNN
+	1    7275 7050
+	0    1    1    0
+$EndComp
+Wire Wire Line
+	7025 7050 7125 7050
+$Comp
+L GND #PWR?
+U 1 1 595EDB7D
+P 7275 7225
+F 0 "#PWR?" H 7275 6975 50  0001 C CNN
+F 1 "GND" H 7280 7052 50  0000 C CNN
+F 2 "" H 7275 7225 50  0001 C CNN
+F 3 "" H 7275 7225 50  0001 C CNN
+	1    7275 7225
+	1    0    0    -1
+$EndComp
+Wire Wire Line
+	7275 7225 7275 7200
+$Comp
+L GND #PWR?
+U 1 1 595EDBF6
+P 6875 7225
+F 0 "#PWR?" H 6875 6975 50  0001 C CNN
+F 1 "GND" H 6880 7052 50  0000 C CNN
+F 2 "" H 6875 7225 50  0001 C CNN
+F 3 "" H 6875 7225 50  0001 C CNN
+	1    6875 7225
+	1    0    0    -1
+$EndComp
+Wire Wire Line
+	6875 7225 6875 7200
+$Comp
+L PE42421 U?
+U 1 1 595EE17B
+P 5950 6850
+F 0 "U?" H 5650 7250 60  0000 R CNN
+F 1 "PE42421" H 6500 7250 60  0000 R CNN
+F 2 "" H 6450 7100 60  0001 C CNN
+F 3 "" H 6450 7100 60  0001 C CNN
+	1    5950 6850
+	1    0    0    -1
+$EndComp
+Wire Wire Line
+	6450 7050 6725 7050
+$Comp
+L PE42421 U?
+U 1 1 595EEAB1
+P 8150 6850
+F 0 "U?" H 7850 7250 60  0000 R CNN
+F 1 "PE42421" H 8700 7250 60  0000 R CNN
+F 2 "" H 8650 7100 60  0001 C CNN
+F 3 "" H 8650 7100 60  0001 C CNN
+	1    8150 6850
+	-1   0    0    -1
+$EndComp
+Wire Wire Line
+	7425 7050 7650 7050
+Wire Wire Line
+	6450 6650 7650 6650
+$Comp
+L GND #PWR?
+U 1 1 595F18F2
+P 5950 7325
+F 0 "#PWR?" H 5950 7075 50  0001 C CNN
+F 1 "GND" H 5955 7152 50  0000 C CNN
+F 2 "" H 5950 7325 50  0001 C CNN
+F 3 "" H 5950 7325 50  0001 C CNN
+	1    5950 7325
+	1    0    0    -1
+$EndComp
+Wire Wire Line
+	5950 7325 5950 7300
+$Comp
+L GND #PWR?
+U 1 1 595F1905
+P 8150 7325
+F 0 "#PWR?" H 8150 7075 50  0001 C CNN
+F 1 "GND" H 8155 7152 50  0000 C CNN
+F 2 "" H 8150 7325 50  0001 C CNN
+F 3 "" H 8150 7325 50  0001 C CNN
+	1    8150 7325
+	1    0    0    -1
+$EndComp
+Wire Wire Line
+	8150 7325 8150 7300
 $EndSCHEMATC

Commit message: Update schematic
Parts:
- removed U?: SAMD20G18A-MU, QFN48, symbol SAMD20G18A-MU
- added AE?: Antenna, symbol Antenna
- added AT? (x3): 10dB, symbol ATTENUATOR
- added C? (x7): C, symbol C
- added J?: CONN_COAXIAL, symbol CONN_COAXIAL
- added U?: SAMD20J18A-MU, QFN64, symbol SAMD20J18A-MU
- added U?: PE42421, symbol PE42421
Connections:
- net labels added: I2C_SCL, I2C_SDA, I2S_FS, I2S_MCK, I2S_SCK, SPI_0_MISO, SPI_0_MOSI, SPI_0_SCK, UART_RX, UART_TX, USB_D+, USB_D-
- wire segments 8 -> 81
Other:
- moved on the sheet: AT?, U?
