File: Hardware/KiCad/FritzRT_MCU/FritzRT_MCU.sch (KiCad schematic (older format))
At the start: 19 parts

Commit message: Schematic work
Parts:
- added C? (x2): C, symbol C
- added U?: Oscillator, symbol Oscillator
Connections:
- net labels added: SPI_1_MISO, SPI_1_MOSI, SPI_1_SCK
- wire segments 81 -> 90
- no-connect marks 0 -> 1
Other:
- moved on the sheet: AT?
Changed lines of the file:
@@
 LIBS:FritzLib2
 LIBS:FritzRT-cache
-EELAYER 25 0
+EELAYER 26 0
 EELAYER END
 $Descr A3 16535 11693
@@
 Text Label 5150 4350 0    47   ~ 0
 USB_D-
-Text Label 5150 2050 0    47   ~ 0
+Text Label 5150 3250 0    47   ~ 0
 UART_RX
-Text Label 5150 1950 0    47   ~ 0
+Text Label 5150 3150 0    47   ~ 0
 UART_TX
-Text Label 5150 3150 0    47   ~ 0
+Text Label 5150 3550 0    47   ~ 0
 SPI_0_MOSI
-Text Label 5150 3250 0    47   ~ 0
+Text Label 5150 3850 0    47   ~ 0
 SPI_0_SCK
-Text Label 5150 3350 0    47   ~ 0
+Text Label 5150 3750 0    47   ~ 0
 SPI_0_MISO
 Text Label 5150 3050 0    47   ~ 0
@@
 Text Label 5150 2950 0    47   ~ 0
 I2S_SCK
+Text Label 1025 4250 0    47   ~ 0
+I2C_SCL
+Text Label 1025 4150 0    47   ~ 0
+I2C_SDA
 Text Label 5150 2850 0    47   ~ 0
-I2C_SCL
-Text Label 5150 2750 0    47   ~ 0
-I2C_SDA
-Text Label 1050 3850 0    47   ~ 0
 I2S_MCK
 Wire Wire Line
@@
 L ATTENUATOR AT?
 U 1 1 5966C641
-P 14675 7300
-F 0 "AT?" V 14468 7300 50  0000 C CNN
-F 1 "10dB" V 14559 7300 50  0000 C CNN
-F 2 "" H 14675 7300 50  0001 C CNN
-F 3 "" H 14675 7300 50  0001 C CNN
-	1    14675 7300
+P 14750 7300
+F 0 "AT?" V 14543 7300 50  0000 C CNN
+F 1 "10dB" V 14634 7300 50  0000 C CNN
+F 2 "" H 14750 7300 50  0001 C CNN
+F 3 "" H 14750 7300 50  0001 C CNN
+	1    14750 7300
 	0    -1   1    0
 $EndComp
@@
 L ATTENUATOR AT?
 U 1 1 5966C647
-P 14275 7300
-F 0 "AT?" V 14068 7300 50  0000 C CNN
-F 1 "10dB" V 14159 7300 50  0000 C CNN
-F 2 "" H 14275 7300 50  0001 C CNN
-F 3 "" H 14275 7300 50  0001 C CNN
-	1    14275 7300
-	0    -1   1    0
-$EndComp
-Wire Wire Line
-	14525 7300 14425 7300
+P 14350 7300
+F 0 "AT?" V 14143 7300 50  0000 C CNN
+F 1 "10dB" V 14234 7300 50  0000 C CNN
+F 2 "" H 14350 7300 50  0001 C CNN
+F 3 "" H 14350 7300 50  0001 C CNN
+	1    14350 7300
+	0    -1   1    0
+$EndComp
+Wire Wire Line
+	14600 7300 14500 7300
 $Comp
 L GND #PWR?
 U 1 1 5966C64E
-P 14275 7625
-F 0 "#PWR?" H 14275 7375 50  0001 C CNN
-F 1 "GND" H 14280 7452 50  0000 C CNN
-F 2 "" H 14275 7625 50  0001 C CNN
-F 3 "" H 14275 7625 50  0001 C CNN
-	1    14275 7625
-	-1   0    0    -1
-$EndComp
-Wire Wire Line
-	14275 7625 14275 7450
+P 14350 7625
+F 0 "#PWR?" H 14350 7375 50  0001 C CNN
+F 1 "GND" H 14355 7452 50  0000 C CNN
+F 2 "" H 14350 7625 50  0001 C CNN
+F 3 "" H 14350 7625 50  0001 C CNN
+	1    14350 7625
+	-1   0    0    -1
+$EndComp
+Wire Wire Line
+	14350 7625 14350 7450
 $Comp
 L GND #PWR?
 U 1 1 5966C655
-P 14675 7625
-F 0 "#PWR?" H 14675 7375 50  0001 C CNN
-F 1 "GND" H 14680 7452 50  0000 C CNN
-F 2 "" H 14675 7625 50  0001 C CNN
-F 3 "" H 14675 7625 50  0001 C CNN
-	1    14675 7625
-	-1   0    0    -1
-$EndComp
-Wire Wire Line
-	14675 7625 14675 7450
-Wire Wire Line
-	15025 7300 14825 7300
+P 14750 7625
+F 0 "#PWR?" H 14750 7375 50  0001 C CNN
+F 1 "GND" H 14755 7452 50  0000 C CNN
+F 2 "" H 14750 7625 50  0001 C CNN
+F 3 "" H 14750 7625 50  0001 C CNN
+	1    14750 7625
+	-1   0    0    -1
+$EndComp
+Wire Wire Line
+	14750 7625 14750 7450
+Wire Wire Line
+	15025 7300 14900 7300
 $Comp
 L ATTENUATOR AT?
 U 1 1 5966C963
-P 13875 7300
-F 0 "AT?" V 13668 7300 50  0000 C CNN
-F 1 "10dB" V 13759 7300 50  0000 C CNN
-F 2 "" H 13875 7300 50  0001 C CNN
-F 3 "" H 13875 7300 50  0001 C CNN
-	1    13875 7300
-	0    -1   1    0
-$EndComp
-Wire Wire Line
-	14125 7300 14025 7300
+P 13950 7300
+F 0 "AT?" V 13743 7300 50  0000 C CNN
+F 1 "10dB" V 13834 7300 50  0000 C CNN
+F 2 "" H 13950 7300 50  0001 C CNN
+F 3 "" H 13950 7300 50  0001 C CNN
+	1    13950 7300
+	0    -1   1    0
+$EndComp
+Wire Wire Line
+	14200 7300 14100 7300
 $Comp
 L GND #PWR?
 U 1 1 5966C96A
-P 13875 7625
-F 0 "#PWR?" H 13875 7375 50  0001 C CNN
-F 1 "GND" H 13880 7452 50  0000 C CNN
-F 2 "" H 13875 7625 50  0001 C CNN
-F 3 "" H 13875 7625 50  0001 C CNN
-	1    13875 7625
-	-1   0    0    -1
-$EndComp
-Wire Wire Line
-	13875 7625 13875 7450
-Wire Wire Line
-	13650 7300 13725 7300
+P 13950 7625
+F 0 "#PWR?" H 13950 7375 50  0001 C CNN
+F 1 "GND" H 13955 7452 50  0000 C CNN
+F 2 "" H 13950 7625 50  0001 C CNN
+F 3 "" H 13950 7625 50  0001 C CNN
+	1    13950 7625
+	-1   0    0    -1
+$EndComp
+Wire Wire Line
+	13950 7625 13950 7450
+Wire Wire Line
+	13650 7300 13800 7300
 $Comp
 L C C?
@@
 Wire Wire Line
 	11150 7300 11200 7300
+Text Label 5150 2350 0    47   ~ 0
+SPI_1_MOSI
+Text Label 5150 2450 0    47   ~ 0
+SPI_1_SCK
+Text Label 5150 2550 0    47   ~ 0
+SPI_1_MISO
+$Comp
+L Oscillator U?
+U 1 1 596DF5A8
+P 5500 9475
+F 0 "U?" H 5225 9775 47  0000 L CNN
+F 1 "Oscillator" H 5600 9775 47  0000 L CNN
+F 2 "" H 5550 9925 47  0001 C CNN
+F 3 "" H 5550 9925 47  0001 C CNN
+	1    5500 9475
+	1    0    0    -1
+$EndComp
+Wire Wire Line
+	6300 8250 6300 9475
+Wire Wire Line
+	6300 9475 5850 9475
+NoConn ~ 6400 8250
+$Comp
+L C C?
+U 1 1 596E08C5
+P 7600 5700
+F 0 "C?" H 7715 5746 50  0000 L CNN
+F 1 "C" H 7715 5655 50  0000 L CNN
+F 2 "" H 7638 5550 50  0001 C CNN
+F 3 "" H 7600 5700 50  0001 C CNN
+	1    7600 5700
+	1    0    0    -1
+$EndComp
+$Comp
+L C C?
+U 1 1 596E0A87
+P 7950 5700
+F 0 "C?" H 8065 5746 50  0000 L CNN
+F 1 "C" H 8065 5655 50  0000 L CNN
+F 2 "" H 7988 5550 50  0001 C CNN
+F 3 "" H 7950 5700 50  0001 C CNN
+	1    7950 5700
+	1    0    0    -1
+$EndComp
+Wire Wire Line
+	7350 6200 7350 5500
+Wire Wire Line
+	7350 5500 7950 5500
+Wire Wire Line
+	7950 5500 7950 5550
+Wire Wire Line
+	7600 5550 7600 5500
+Connection ~ 7600 5500
+$Comp
+L GND #PWR?
+U 1 1 596E10D4
+P 7950 5900
+F 0 "#PWR?" H 7950 5650 50  0001 C CNN
+F 1 "GND" H 7955 5727 50  0000 C CNN
+F 2 "" H 7950 5900 50  0001 C CNN
+F 3 "" H 7950 5900 50  0001 C CNN
+	1    7950 5900
+	1    0    0    -1
+$EndComp
+Wire Wire Line
+	7950 5900 7950 5850
+Wire Wire Line
+	7950 5875 7600 5875
+Wire Wire Line
+	7600 5875 7600 5850
+Connection ~ 7950 5875
 $EndSCHEMATC
