File: Hardware/KiCad/FritzRT_RF/FritzRT_RF.sch (KiCad schematic (older format))
At the start: 49 parts

Commit message: schematic work
Parts:
- removed AT?: 10dB, symbol ATTENUATOR
- removed C? (x6): C, symbol C
- removed R?: R, symbol R
- removed U?: Oscillator, symbol Oscillator
- removed U?: DC09-73LF, symbol DC09-73LF
- removed U?: LMV221, symbol LMV221
- added C? (x9): C, symbol C
- added C? (x4): 100nF, symbol C
- added C?: 10uF, symbol C
- added J?: CONN_02X16, symbol CONN_02X16
- added R? (x6): 1k, symbol R
- added R? (x5): 27R, symbol R
- added Y?: Crystal, symbol Crystal
Connections:
- net +3V3: now also U?.13 (VBAT1), U?.27 (VBAT2), C?.1, C?.1, C?.1, C?.1, C?.1, J?.2 (P2), J?.4 (P4), R?.1, R?.1, R?.1
- net GND: now also C?.1, C?.1, C?.2, C?.2, C?.2, C?.2, C?.2, C?.2, C?.2, C?.2, J?.1 (P1), J?.11 (P11), J?.13 (P13), J?.15 (P15), J?.17 (P17), J?.19 (P19), J?.21 (P21), J?.23 (P23), J?.25 (P25), J?.27 (P27), J?.29 (P29), J?.3 (P3), J?.31 (P31), J?.5 (P5), J?.7 (P7), J?.9 (P9)
- net at U?.15 (VR_ANA): now also C?.1
- net at U?.16 (VR_DIG): now also C?.1
- net at U?.17 (XTA): now also C?.2, Y?.1
- net at U?.18 (XTB): now also C?.2, Y?.2
- net ~RESET: now reaches U?.19 (RESET)
- net ~RESET: now also J?.8 (P8)
- net DIO0: now reaches U?.21 (DIO0)
- net DIO0: now also J?.10 (P10)
- net at U?.22 (DIO1/DCLK): now also R?.1
- net at U?.23 (DIO2/DATA): now also R?.1
- net DIO3: now reaches U?.24 (DIO3)
- net DIO3: now also J?.16 (P16)
- net DIO4: now reaches U?.25 (DIO4)
- net DIO4: now also J?.18 (P18)
- net DIO5: now reaches U?.26 (DIO5)
- net DIO5: now also J?.20 (P20)
- net at U?.29 (SCK): now also R?.1
- net at U?.30 (MISO): now also R?.1
- net at U?.31 (MOSI): now also R?.1
- net ~CS: now reaches U?.32 (NSS)
- net ~CS: now also J?.28 (P28)
- net ~RX~/TX: now reaches U?.8 (RXTX)
- net ~RX~/TX: now also J?.6 (P6)
- net at U?.3 (RF2): now also C?.2
- net at U?.4 (CTRL): now also R?.2 (x3)
- net at U?.5 (RFC): now also C?.1
- net at U?.6 (~CTRL~/VDD): now also R?.2 (x3)
- net at U?.3 (RF2): now also C?.1
- net at U?.5 (RFC): now also C?.2
- net at AE?.1 (A), C?.2, L?.1: now also C?.2
- net at C?.2, J?.1 (In), L?.1: now also C?.2
- net at L?.2: now also C?.1 (x2)
- new net ANT/~EXT~: J?.30 (P30), R?.1
- new net DIO1/CLK: J?.12 (P12), R?.2
- new net DIO2/DATA: J?.14 (P14), R?.2
- new net MISO: J?.24 (P24), R?.2
- new net MOSI: J?.26 (P26), R?.2
- new net PASS/~TNDWN~: J?.32 (P32), R?.1, R?.1
- new net SCK: J?.22 (P22), R?.2
- no-connect marks 2 -> 1
Other:
- moved on the sheet: AE?, AT?, C?, J?, L?, R?, U?

Commit message: Updated connector and antenna P/Ns
Parts:
- AE?: value Antenna -> ANT1204LL05R0915A
- C? (x4): value C -> 120pF
- C? (x2): value C -> 50pF
- J?: value CONN_COAXIAL -> CON-SMA-EDGE-S
- L? (x4): value L -> 200nH
- L? (x2): value L -> 620uH
Changed lines of the file:
@@
 P 10850 7950
 F 0 "AE?" H 10775 8025 50  0000 R CNN
-F 1 "Antenna" H 10775 7950 50  0000 R CNN
+F 1 "ANT1204LL05R0915A" H 10775 7950 50  0000 R CNN
 F 2 "" H 10850 7950 50  0001 C CNN
 F 3 "" H 10850 7950 50  0001 C CNN
@@
 U 1 1 5966B9DA
 P 10850 9350
-F 0 "J?" H 10860 9470 50  0000 C CNN
-F 1 "CONN_COAXIAL" V 10965 9350 50  0000 C CNN
+F 0 "J?" H 11000 9400 50  0000 C CNN
+F 1 "CON-SMA-EDGE-S" H 11300 9300 50  0000 C CNN
 F 2 "" H 10850 9350 50  0001 C CNN
 F 3 "" H 10850 9350 50  0001 C CNN
@@
 P 8900 9550
 F 0 "C?" H 9100 9500 50  0000 R CNN
-F 1 "C" H 9100 9600 50  0000 R CNN
+F 1 "120pF" H 9250 9600 50  0000 R CNN
 F 2 "" H 8938 9400 50  0001 C CNN
 F 3 "" H 8900 9550 50  0001 C CNN
@@
 P 9100 9550
 F 0 "L?" H 9153 9596 50  0000 L CNN
-F 1 "L" H 9153 9505 50  0000 L CNN
+F 1 "200nH" H 9153 9505 50  0000 L CNN
 F 2 "" H 9100 9550 50  0001 C CNN
 F 3 "" H 9100 9550 50  0001 C CNN
@@
 P 9400 9350
 F 0 "L?" V 9590 9350 50  0000 C CNN
-F 1 "L" V 9499 9350 50  0000 C CNN
+F 1 "620uH" V 9499 9350 50  0000 C CNN
 F 2 "" H 9400 9350 50  0001 C CNN
 F 3 "" H 9400 9350 50  0001 C CNN
@@
 P 10100 9550
 F 0 "C?" H 10300 9500 50  0000 R CNN
-F 1 "C" H 10300 9600 50  0000 R CNN
+F 1 "120pF" H 10450 9600 50  0000 R CNN
 F 2 "" H 10138 9400 50  0001 C CNN
 F 3 "" H 10100 9550 50  0001 C CNN
@@
 P 10300 9550
 F 0 "L?" H 10353 9596 50  0000 L CNN
-F 1 "L" H 10353 9505 50  0000 L CNN
+F 1 "200nH" H 10353 9505 50  0000 L CNN
 F 2 "" H 10300 9550 50  0001 C CNN
 F 3 "" H 10300 9550 50  0001 C CNN
@@
 P 8900 8600
 F 0 "C?" H 9100 8550 50  0000 R CNN
-F 1 "C" H 9100 8650 50  0000 R CNN
+F 1 "120pF" H 9250 8650 50  0000 R CNN
 F 2 "" H 8938 8450 50  0001 C CNN
 F 3 "" H 8900 8600 50  0001 C CNN
@@
 P 9100 8600
 F 0 "L?" H 9153 8646 50  0000 L CNN
-F 1 "L" H 9153 8555 50  0000 L CNN
+F 1 "200nH" H 9153 8555 50  0000 L CNN
 F 2 "" H 9100 8600 50  0001 C CNN
 F 3 "" H 9100 8600 50  0001 C CNN
@@
 P 9400 8400
 F 0 "L?" V 9590 8400 50  0000 C CNN
-F 1 "L" V 9499 8400 50  0000 C CNN
+F 1 "620uH" V 9499 8400 50  0000 C CNN
 F 2 "" H 9400 8400 50  0001 C CNN
 F 3 "" H 9400 8400 50  0001 C CNN
@@
 P 10100 8600
 F 0 "C?" H 10300 8550 50  0000 R CNN
-F 1 "C" H 10300 8650 50  0000 R CNN
+F 1 "120pF" H 10450 8650 50  0000 R CNN
 F 2 "" H 10138 8450 50  0001 C CNN
 F 3 "" H 10100 8600 50  0001 C CNN
@@
 P 10300 8600
 F 0 "L?" H 10353 8646 50  0000 L CNN
-F 1 "L" H 10353 8555 50  0000 L CNN
+F 1 "200nH" H 10353 8555 50  0000 L CNN
 F 2 "" H 10300 8600 50  0001 C CNN
 F 3 "" H 10300 8600 50  0001 C CNN
@@
 P 9750 8400
 F 0 "C?" V 9500 8350 50  0000 L CNN
-F 1 "C" V 9600 8300 50  0000 L CNN
+F 1 "50pF" V 9600 8300 50  0000 L CNN
 F 2 "" H 9788 8250 50  0001 C CNN
 F 3 "" H 9750 8400 50  0001 C CNN
@@
 P 9750 9350
 F 0 "C?" V 9500 9300 50  0000 L CNN
-F 1 "C" V 9600 9250 50  0000 L CNN
+F 1 "50pF" V 9600 9250 50  0000 L CNN
 F 2 "" H 9788 9200 50  0001 C CNN
 F 3 "" H 9750 9350 50  0001 C CNN
@@
 	5350 8800 5500 8800
 Wire Wire Line
-	13675 1325 13850 1325
-Wire Wire Line
-	13850 1325 14275 1325
-Wire Wire Line
-	14275 1275 14275 1325
-Wire Wire Line
-	14275 1325 14275 1375
+	13675 1325 14275 1325
+Wire Wire Line
+	14275 1275 14275 1375
 Wire Wire Line
 	13850 1375 13850 1325
 Connection ~ 13850 1325
 Wire Wire Line
-	14275 1675 14275 1700
-Wire Wire Line
-	14275 1700 14275 1725
+	14275 1675 14275 1725
 Wire Wire Line
 	14275 1700 13850 1700
@@
 	11050 4050 11050 4025
 Wire Wire Line
-	11050 4025 11150 4025
-Wire Wire Line
-	11150 4025 11250 4025
-Wire Wire Line
-	11250 4025 11350 4025
-Wire Wire Line
-	11350 4025 11450 4025
-Wire Wire Line
-	11450 4025 11550 4025
-Wire Wire Line
-	11550 4025 11650 4025
+	11050 4025 11650 4025
 Wire Wire Line
 	11650 4025 11650 4000
@@
 Connection ~ 11150 4025
 Wire Wire Line
-	13150 4525 13150 4575
-Wire Wire Line
-	13150 4575 13150 4600
+	13150 4525 13150 4600
 Wire Wire Line
 	13150 4575 13550 4575
 Wire Wire Line
-	13550 4550 13550 4575
-Wire Wire Line
-	13550 4575 13550 4600
+	13550 4550 13550 4600
 Connection ~ 13150 4575
 Wire Wire Line
-	13550 4900 13550 4925
-Wire Wire Line
-	13550 4925 13550 4950
+	13550 4900 13550 4950
 Wire Wire Line
 	13550 4925 13150 4925
@@
 	13950 4575 14350 4575
 Wire Wire Line
-	14350 4550 14350 4575
-Wire Wire Line
-	14350 4575 14350 4600
+	14350 4550 14350 4600
 Connection ~ 13950 4575
 Wire Wire Line
-	14350 4900 14350 4925
-Wire Wire Line
-	14350 4925 14350 4950
+	14350 4900 14350 4950
 Wire Wire Line
 	14350 4925 13950 4925
@@
 Connection ~ 13550 4575
 Wire Wire Line
-	13950 4075 13950 4575
-Wire Wire Line
-	13950 4575 13950 4600
+	13950 4075 13950 4600
 Connection ~ 14350 4575
 Wire Wire Line
@@
 	12600 1150 12600 1200
 Wire Wire Line
-	11900 1150 12250 1150
-Wire Wire Line
-	12250 1150 12600 1150
+	11900 1150 12600 1150
 Wire Wire Line
 	11900 1150 11900 1200
@@
 	11900 1550 11900 1500
 Wire Wire Line
-	10625 5525 10800 5525
-Wire Wire Line
-	10800 5525 10950 5525
+	10625 5525 10950 5525
 Wire Wire Line
 	10325 5525 10125 5525
 Wire Wire Line
-	10125 4975 10125 5525
-Wire Wire Line
-	10125 5525 10125 5550
+	10125 4975 10125 5550
 Wire Wire Line
 	11250 5525 11325 5525
 Wire Wire Line
-	11625 5525 11775 5525
-Wire Wire Line
-	11775 5525 11975 5525
+	11625 5525 11975 5525
 Wire Wire Line
 	11775 5525 11775 5550
@@
 	12275 5525 12450 5525
 Wire Wire Line
-	12450 4000 12450 5525
-Wire Wire Line
-	12450 5525 12450 5550
+	12450 4000 12450 5550
 Wire Wire Line
 	12450 5900 12450 5850
@@
 	8900 9400 8900 9350
 Wire Wire Line
-	8500 9350 8900 9350
-Wire Wire Line
-	8900 9350 9100 9350
-Wire Wire Line
-	9100 9350 9250 9350
+	8500 9350 9250 9350
 Wire Wire Line
 	9100 9400 9100 9350
@@
 	8900 9700 8900 9750
 Wire Wire Line
-	8900 9750 9000 9750
-Wire Wire Line
-	9000 9750 9100 9750
+	8900 9750 9100 9750
 Wire Wire Line
 	9100 9750 9100 9700
@@
 	10100 9400 10100 9350
 Wire Wire Line
-	9900 9350 10100 9350
-Wire Wire Line
-	10100 9350 10300 9350
-Wire Wire Line
-	10300 9350 10700 9350
+	9900 9350 10700 9350
 Wire Wire Line
 	10300 9350 10300 9400
@@
 	10100 9700 10100 9750
 Wire Wire Line
-	10100 9750 10200 9750
-Wire Wire Line
-	10200 9750 10300 9750
+	10100 9750 10300 9750
 Wire Wire Line
 	10300 9750 10300 9700
@@
 	8900 8450 8900 8400
 Wire Wire Line
-	8300 8400 8900 8400
-Wire Wire Line
-	8900 8400 9100 8400
-Wire Wire Line
-	9100 8400 9250 8400
+	8300 8400 9250 8400
 Wire Wire Line
 	9100 8450 9100 8400
@@
 	8900 8750 8900 8800
 Wire Wire Line
-	8900 8800 9000 8800
-Wire Wire Line
-	9000 8800 9100 8800
+	8900 8800 9100 8800
 Wire Wire Line
 	9100 8800 9100 8750
@@
 	10100 8450 10100 8400
 Wire Wire Line
-	9900 8400 10100 8400
-Wire Wire Line
-	10100 8400 10300 8400
-Wire Wire Line
-	10300 8400 10850 8400
+	9900 8400 10850 8400
 Wire Wire Line
 	10300 8400 10300 8450
@@
 	10100 8750 10100 8800
 Wire Wire Line
-	10100 8800 10200 8800
-Wire Wire Line
-	10200 8800 10300 8800
+	10100 8800 10300 8800
 Wire Wire Line
 	10300 8800 10300 8750
@@
 	11850 4350 11850 4000
 Wire Wire Line
-	9100 4350 9450 4350
-Wire Wire Line
-	9450 4350 11850 4350
+	9100 4350 11850 4350
 Wire Wire Line
 	9450 4350 9450 4400
@@
 	11950 4750 11950 4000
 Wire Wire Line
-	9100 4750 9450 4750
-Wire Wire Line
-	9450 4750 11950 4750
+	9100 4750 11950 4750
 Wire Wire Line
 	9450 4750 9450 4700
@@
 	8800 4350 8650 4350
 Wire Wire Line
-	8650 4350 8650 4750
-Wire Wire Line
-	8650 4750 8650 4850
+	8650 4350 8650 4850
 Wire Wire Line
 	8800 4750 8650 4750
@@
 	3500 8100 3500 8150
 Wire Wire Line
-	3400 7100 3400 7300
-Wire Wire Line
-	3400 7300 3400 7800
-Wire Wire Line
-	6050 7100 6050 7300
-Wire Wire Line
-	6050 7300 6050 7800
-Wire Wire Line
-	7750 7100 7750 7300
-Wire Wire Line
-	7750 7300 7750 7800
+	3400 7100 3400 7800
+Wire Wire Line
+	6050 7100 6050 7800
+Wire Wire Line
+	7750 7100 7750 7800
 Wire Wire Line
 	3500 7800 3500 7700
 Wire Wire Line
-	900  7700 3500 7700
-Wire Wire Line
-	3500 7700 5950 7700
+	900  7700 5950 7700
 Wire Wire Line
 	5950 7700 5950 7800
@@
 	9800 1150 9800 1400
 Wire Wire Line
-	8900 1150 9350 1150
-Wire Wire Line
-	9350 1150 11500 1150
-Wire Wire Line
-	11500 1150 11500 1900
-Wire Wire Line
-	11500 1900 11500 1950
+	8900 1150 11500 1150
+Wire Wire Line
+	11500 1150 11500 1950
 Wire Wire Line
 	11600 1950 11600 1900
@@
 Connection ~ 11500 1900
 Wire Wire Line
-	8900 1050 8900 1150
-Wire Wire Line
-	8900 1150 8900 1400
+	8900 1050 8900 1400
 Wire Wire Line
 	9350 1150 9350 1400
@@
 	9350 1700 9350 1750
 Wire Wire Line
-	8900 1750 9350 1750
-Wire Wire Line
-	9350 1750 9800 1750
+	8900 1750 9800 1750
 Wire Wire Line
 	10300 1750 10750 1750
@@
 Connection ~ 9350 1750
 Wire Wire Line
-	10300 1700 10300 1750
-Wire Wire Line
-	10300 1750 10300 1800
+	10300 1700 10300 1800
 Connection ~ 10300 1750
 Wire Wire Line
@@
 $EndComp
 Wire Wire Line
-	5350 2650 5350 2750
-Wire Wire Line
-	5350 2750 5350 2850
-Wire Wire Line
-	5350 2850 5350 2950
-Wire Wire Line
-	5350 2950 5350 3050
-Wire Wire Line
-	5350 3050 5350 3150
-Wire Wire Line
-	5350 3150 5350 3250
-Wire Wire Line
-	5350 3250 5350 3350
-Wire Wire Line
-	5350 3350 5350 3450
-Wire Wire Line
-	5350 3450 5350 3550
-Wire Wire Line
-	5350 3550 5350 3650
-Wire Wire Line
-	5350 3650 5350 3750
-Wire Wire Line
-	5350 3750 5350 3850
-Wire Wire Line
-	5350 3850 5350 3950
-Wire Wire Line
-	5350 3950 5350 4050
-Wire Wire Line
-	5350 4050 5350 4150
-Wire Wire Line
-	5350 4150 5350 4250
+	5350 2650 5350 4250
 Wire Wire Line
 	5350 2850 5450 2850
@@
 $EndComp
 Wire Wire Line
-	6400 2550 6400 2650
-Wire Wire Line
-	6400 2650 6400 2750
+	6400 2550 6400 2750
 Wire Wire Line
 	6400 2750 5950 2750
@@
 	8550 2150 8650 2250
 Wire Wire Line
-	8900 1700 8900 1750
-Wire Wire Line
-	8900 1750 8900 1800
+	8900 1700 8900 1800
 $Comp
 L C C?
@@
 $EndComp
 Connection ~ 8900 1750
+Wire Bus Line
+	8550 3550 8550 2150
+Wire Bus Line
+	6600 4050 6600 2750
+Entry Wire Line
+	800  7600 900  7700
+Entry Wire Line
+	800  7500 900  7600
+Wire Bus Line
+	800  7600 800  7500
 $EndSCHEMATC

Commit message: Created SX1238 Board bringup project
Parts:
- L? (x2): value 620uH -> 620nH
Changed lines of the file:
@@
 P 9400 9350
 F 0 "L?" V 9590 9350 50  0000 C CNN
-F 1 "620uH" V 9499 9350 50  0000 C CNN
+F 1 "620nH" V 9499 9350 50  0000 C CNN
 F 2 "" H 9400 9350 50  0001 C CNN
 F 3 "" H 9400 9350 50  0001 C CNN
@@
 P 9400 8400
 F 0 "L?" V 9590 8400 50  0000 C CNN
-F 1 "620uH" V 9499 8400 50  0000 C CNN
+F 1 "620nH" V 9499 8400 50  0000 C CNN
 F 2 "" H 9400 8400 50  0001 C CNN
 F 3 "" H 9400 8400 50  0001 C CNN
